File: eagle/uPy_AudioCodec_00.sch (EAGLE design)
At the start: 42 parts, among them J1 TSW-108-02-S-S-MOD, J2 TSW-108-02-S-S-MOD, U1 SSM2604-1, U3 TPA6130A2

Commit message: Directory reorganization: eagle files moved to eagle/, pdf files moved to docs/, add gerber files
Parts:
- C14, C17, C20, C21: value 220pF -> 150pF
Changed lines of the file:
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@@
 <part name="P+1" library="supply1" deviceset="+5V" device=""/>
 <part name="SUPPLY6" library="supply2" deviceset="GND" device=""/>
-<part name="C14" library="rcl" deviceset="C-US" device="C0603K" value="220pF"/>
-<part name="C17" library="rcl" deviceset="C-US" device="C0603K" value="220pF"/>
+<part name="C14" library="rcl" deviceset="C-US" device="C0603K" value="150pF"/>
+<part name="C17" library="rcl" deviceset="C-US" device="C0603K" value="150pF"/>
 <part name="R1" library="rcl" deviceset="R-US_" device="R0805" value="4.99K"/>
 <part name="R2" library="rcl" deviceset="R-US_" device="R0805" value="4.99K"/>
@@
 <part name="R3" library="rcl" deviceset="R-US_" device="R0805" value="4.99K"/>
 <part name="R4" library="rcl" deviceset="R-US_" device="R0805" value="4.99K"/>
-<part name="C20" library="rcl" deviceset="C-US" device="C0603K" value="220pF"/>
-<part name="C21" library="rcl" deviceset="C-US" device="C0603K" value="220pF"/>
+<part name="C20" library="rcl" deviceset="C-US" device="C0603K" value="150pF"/>
+<part name="C21" library="rcl" deviceset="C-US" device="C0603K" value="150pF"/>
 <part name="L2" library="rcl" deviceset="L-US" device="L3216C"/>
 <part name="L3" library="rcl" deviceset="L-US" device="L3216C"/>
